Commit message: 添加位姿透传遥操作模式

File: rml63_teleop/assets/rml63/robot_full.urdf (robot description, URDF)
Before this commit: robot my_robot, 15 links, 14 joints
Links:
- removed link link1
- removed link link2
- removed link link3
- removed link link4
- removed link link5
- removed link link6
- added link camera_link, mass 9.2946E-05; collision mesh filename=../rm_models/RML63/urdf/RML63II/RML63II-6F-V/meshes/camera_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; visual mesh filename=../rm_models/RML63/urdf/RML63II/RML63II-6F-V/meshes/camera_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
- added link camera_rolink, mass 0.21281; collision mesh filename=../rm_models/RML63/urdf/RML63II/RML63II-6F-V/meshes/camera_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; visual mesh filename=../rm_models/RML63/urdf/RML63II/RML63II-6F-V/meshes/camera_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
- added link connector_link; collision cylinder length=0.076 radius=0.029; visual cylinder length=0.076 radius=0.029
- added link link_1, mass 1.837; collision mesh filename=../rm_models/RML63/urdf/RML63II/RML63II-6F-V/meshes/link_1.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; visual mesh filename=../rm_models/RML63/urdf/RML63II/RML63II-6F-V/meshes/link_1.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
- added link link_2, mass 2.006; collision mesh filename=../rm_models/RML63/urdf/RML63II/RML63II-6F-V/meshes/link_2.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; visual mesh filename=../rm_models/RML63/urdf/RML63II/RML63II-6F-V/meshes/link_2.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
- added link link_3, mass 1.961; collision mesh filename=../rm_models/RML63/urdf/RML63II/RML63II-6F-V/meshes/link_3.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; visual mesh filename=../rm_models/RML63/urdf/RML63II/RML63II-6F-V/meshes/link_3.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
- added link link_4, mass 1.201; collision mesh filename=../rm_models/RML63/urdf/RML63II/RML63II-6F-V/meshes/link_4.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; visual mesh filename=../rm_models/RML63/urdf/RML63II/RML63II-6F-V/meshes/link_4.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
- added link link_5, mass 1.026; collision mesh filename=../rm_models/RML63/urdf/RML63II/RML63II-6F-V/meshes/link_5.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; visual mesh filename=../rm_models/RML63/urdf/RML63II/RML63II-6F-V/meshes/link_5.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
- added link link_6, mass 0.248; collision mesh filename=../rm_models/RML63/urdf/RML63II/RML63II-6F-V/meshes/link_6.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; visual mesh filename=../rm_models/RML63/urdf/RML63II/RML63II-6F-V/meshes/link_6.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
- link base_link: mass 0.604237569846431 -> 1.862; geometry collision mesh filename=../rm_models/RML63/urdf/RML63II/RML63II-6F-V/meshes/base_li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; visual mesh filename=../rm_models/RML63/urdf/RML63II/RML63II-6F-V/meshes/base_li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
- link gripper_gripper_base: geometry collision mesh filename=../rml63/meshes/EG2-4C2/baselink.obj; visual mesh filename=../rml63/meshes/EG2-4C2/baselink.obj
- link gripper_left_inner_link: geometry collision mesh filename=../rml63/meshes/EG2-4C2/inner_link.obj; visual mesh filename=../rml63/meshes/EG2-4C2/inner_link.obj
- link gripper_left_outer_link: geometry collision mesh filename=../rml63/meshes/EG2-4C2/outer_link.obj; visual mesh filename=../rml63/meshes/EG2-4C2/outer_link.obj
- link gripper_left_pad: geometry collision mesh filename=../rml63/meshes/EG2-4C2/pad.obj; visual mesh filename=../rml63/meshes/EG2-4C2/pad.obj
- link gripper_right_inner_link: geometry collision mesh filename=../rml63/meshes/EG2-4C2/inner_link.obj scale=-1 1 1; visual mesh filename=../rml63/meshes/EG2-4C2/inner_link.obj scale=-1 1 1
- link gripper_right_outer_link: geometry collision mesh filename=../rml63/meshes/EG2-4C2/outer_link.obj scale=-1 1 1; visual mesh filename=../rml63/meshes/EG2-4C2/outer_link.obj scale=-1 1 1
- link gripper_right_pad: geometry collision mesh filename=../rml63/meshes/EG2-4C2/pad.obj scale=-1 1 1; visual mesh filename=../rml63/meshes/EG2-4C2/pad.obj scale=-1 1 1
Joints:
- removed joint joint1
- removed joint joint2
- removed joint joint3
- removed joint joint4
- removed joint joint5
- removed joint joint6
- added joint camera_joint: type fixed, parent camera_rolink, child camera_link, origin xyz=0.02978 -0.0395 -0.0345 rpy=2.0452 1.5708 2.0452
- added joint camera_rojoint: type fixed, parent link_6, child camera_rolink, origin xyz=0.045 -0.002 -0.0653 rpy=-3.1416 -1.5708 -1.5708
- added joint connector_mount: type fixed, parent link_6, child connector_link, origin xyz=0 0 0 rpy=0 0 0
- added joint joint_1: type revolute, parent base_link, child link_1, origin xyz=0 0 0.172 rpy=0 0 0, axis 0 0 1, limit lower=-3.106 upper=3.106 effort=60 velocity=3.14
- added joint joint_2: type revolute, parent link_1, child link_2, origin xyz=-0.086 0 0 rpy=1.5708 -1.5708 3.14, axis 0 0 1, limit lower=-3.106 upper=3.106 effort=60 velocity=3.14
- added joint joint_3: type revolute, parent link_2, child link_3, origin xyz=0.38 0 0 rpy=0 0 1.5708, axis 0 0 1, limit lower=-3.106 upper=2.5307 effort=30 velocity=3.14
- added joint joint_4: type revolute, parent link_3, child link_4, origin xyz=0.069 -0.405 0 rpy=1.5708 0 0, axis 0 0 1, limit lower=-3.106 upper=3.106 effort=30 velocity=3.14
- added joint joint_5: type revolute, parent link_4, child link_5, origin xyz=0 0 0 rpy=1.5708 0 3.1416, axis 0 0 1, limit lower=-3.106 upper=3.106 effort=10 velocity=3.14
- added joint joint_6: type revolute, parent link_5, child link_6, origin xyz=0 0.1666 0 rpy=1.5708 0 3.1416, axis 0 0 1, limit lower=-6.28 upper=6.28 effort=10 velocity=3.14
- joint gripper_mount: origin xyz=0 0 0 rpy=0 0 1.5708 -> xyz=0 0 0.076 rpy=0 0 1.5708; parent link6 -> connector_link

File: rml63_teleop/assets/rml63/robot_ik.urdf (robot description, URDF)
Before this commit: robot my_robot, 15 links, 14 joints
Links:
- removed link link1
- removed link link2
- removed link link3
- removed link link4
- removed link link5
- removed link link6
- added link camera_link, mass 9.2946E-05; collision mesh filename=../rm_models/RML63/urdf/RML63II/RML63II-6F-V/meshes/camera_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; visual mesh filename=../rm_models/RML63/urdf/RML63II/RML63II-6F-V/meshes/camera_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
- added link camera_rolink, mass 0.21281; collision mesh filename=../rm_models/RML63/urdf/RML63II/RML63II-6F-V/meshes/camera_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; visual mesh filename=../rm_models/RML63/urdf/RML63II/RML63II-6F-V/meshes/camera_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
- added link connector_link; collision cylinder length=0.076 radius=0.029; visual cylinder length=0.076 radius=0.029
- added link link_1, mass 1.837; collision mesh filename=../rm_models/RML63/urdf/RML63II/RML63II-6F-V/meshes/link_1.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; visual mesh filename=../rm_models/RML63/urdf/RML63II/RML63II-6F-V/meshes/link_1.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
- added link link_2, mass 2.006; collision mesh filename=../rm_models/RML63/urdf/RML63II/RML63II-6F-V/meshes/link_2.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; visual mesh filename=../rm_models/RML63/urdf/RML63II/RML63II-6F-V/meshes/link_2.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
- added link link_3, mass 1.961; collision mesh filename=../rm_models/RML63/urdf/RML63II/RML63II-6F-V/meshes/link_3.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; visual mesh filename=../rm_models/RML63/urdf/RML63II/RML63II-6F-V/meshes/link_3.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
- added link link_4, mass 1.201; collision mesh filename=../rm_models/RML63/urdf/RML63II/RML63II-6F-V/meshes/link_4.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; visual mesh filename=../rm_models/RML63/urdf/RML63II/RML63II-6F-V/meshes/link_4.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
- added link link_5, mass 1.026; collision mesh filename=../rm_models/RML63/urdf/RML63II/RML63II-6F-V/meshes/link_5.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; visual mesh filename=../rm_models/RML63/urdf/RML63II/RML63II-6F-V/meshes/link_5.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
- added link link_6, mass 0.248; collision mesh filename=../rm_models/RML63/urdf/RML63II/RML63II-6F-V/meshes/link_6.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; visual mesh filename=../rm_models/RML63/urdf/RML63II/RML63II-6F-V/meshes/link_6.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
- link base_link: mass 0.604237569846431 -> 1.862; geometry collision mesh filename=../rm_models/RML63/urdf/RML63II/RML63II-6F-V/meshes/base_li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; visual mesh filename=../rm_models/RML63/urdf/RML63II/RML63II-6F-V/meshes/base_li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
- link gripper_gripper_base: geometry collision mesh filename=../rml63/meshes/EG2-4C2/baselink.obj; visual mesh filename=../rml63/meshes/EG2-4C2/baselink.obj
- link gripper_left_inner_link: geometry collision mesh filename=../rml63/meshes/EG2-4C2/inner_link.obj; visual mesh filename=../rml63/meshes/EG2-4C2/inner_link.obj
- link gripper_left_outer_link: geometry collision mesh filename=../rml63/meshes/EG2-4C2/outer_link.obj; visual mesh filename=../rml63/meshes/EG2-4C2/outer_link.obj
- link gripper_left_pad: geometry collision mesh filename=../rml63/meshes/EG2-4C2/pad.obj; visual mesh filename=../rml63/meshes/EG2-4C2/pad.obj
- link gripper_right_inner_link: geometry collision mesh filename=../rml63/meshes/EG2-4C2/inner_link.obj scale=-1 1 1; visual mesh filename=../rml63/meshes/EG2-4C2/inner_link.obj scale=-1 1 1
- link gripper_right_outer_link: geometry collision mesh filename=../rml63/meshes/EG2-4C2/outer_link.obj scale=-1 1 1; visual mesh filename=../rml63/meshes/EG2-4C2/outer_link.obj scale=-1 1 1
- link gripper_right_pad: geometry collision mesh filename=../rml63/meshes/EG2-4C2/pad.obj scale=-1 1 1; visual mesh filename=../rml63/meshes/EG2-4C2/pad.obj scale=-1 1 1
Joints:
- removed joint joint1
- removed joint joint2
- removed joint joint3
- removed joint joint4
- removed joint joint5
- removed joint joint6
- added joint camera_joint: type fixed, parent camera_rolink, child camera_link, origin xyz=0.02978 -0.0395 -0.0345 rpy=2.0452 1.5708 2.0452
- added joint camera_rojoint: type fixed, parent link_6, child camera_rolink, origin xyz=0.045 -0.002 -0.0653 rpy=-3.1416 -1.5708 -1.5708
- added joint connector_mount: type fixed, parent link_6, child connector_link, origin xyz=0 0 0 rpy=0 0 0
- added joint joint_1: type revolute, parent base_link, child link_1, origin xyz=0 0 0.172 rpy=0 0 0, axis 0 0 1, limit lower=-3.106 upper=3.106 effort=60 velocity=3.14
- added joint joint_2: type revolute, parent link_1, child link_2, origin xyz=-0.086 0 0 rpy=1.5708 -1.5708 3.14, axis 0 0 1, limit lower=-3.106 upper=3.106 effort=60 velocity=3.14
- added joint joint_3: type revolute, parent link_2, child link_3, origin xyz=0.38 0 0 rpy=0 0 1.5708, axis 0 0 1, limit lower=-3.106 upper=2.5307 effort=30 velocity=3.14
- added joint joint_4: type revolute, parent link_3, child link_4, origin xyz=0.069 -0.405 0 rpy=1.5708 0 0, axis 0 0 1, limit lower=-3.106 upper=3.106 effort=30 velocity=3.14
- added joint joint_5: type revolute, parent link_4, child link_5, origin xyz=0 0 0 rpy=1.5708 0 3.1416, axis 0 0 1, limit lower=-3.106 upper=3.106 effort=10 velocity=3.14
- added joint joint_6: type revolute, parent link_5, child link_6, origin xyz=0 0.1666 0 rpy=1.5708 0 3.1416, axis 0 0 1, limit lower=-6.28 upper=6.28 effort=10 velocity=3.14
- joint gripper_mount: origin xyz=0 0 0 rpy=0 0 1.5708 -> xyz=0 0 0.076 rpy=0 0 1.5708; parent link6 -> connector_link
